File: usb.kicad_sch (KiCad schematic)
At the start: 0 parts

Commit message: add decoupling pins
Parts:
- added J1: USB_C_Receptacle_USB2.0_14P, symbol Connector:USB_C_Receptacle_USB2.0_14P
- added R2, R3: 5.1k, symbol Device:R
Connections:
- new net: J1.B5 (CC2), R3.1
- new net: J1.A5 (CC1), R2.1
- new net GND: J1.A1 (GND), J1.A12 (GND), J1.B1 (GND), J1.B12 (GND), J1.SH (SHIELD), R2.2, R3.2
- new net OTG_HS_DM: J1.A7 (D-), J1.B7 (D-)
- new net OTG_HS_DP: J1.A6 (D+), J1.B6 (D+)
- new net VBUS: J1.A4 (VBUS), J1.A9 (VBUS), J1.B4 (VBUS), J1.B9 (VBUS)
Other:
- note added: "USB-C Receptacle"
