File: analog.kicad_sch (KiCad schematic)
At the start: 0 parts

Commit message: add sensors and muxes
Other:
- added sheet bank13 (bank13.kicad_sch)
- added sheet bank16_0 (bank16.kicad_sch)
- added sheet bank16_1 (bank16.kicad_sch)
- added sheet bank16_2 (bank16.kicad_sch)
- added sheet bank16_3 (bank16.kicad_sch)
