File: kicad/RGB.kicad_sch (KiCad schematic)
At the start: 0 parts

Commit message: finish schematics
Parts:
- added C41, C42: 100nF, symbol Device:C
- added R9: 470, symbol Device:R
- added TP1, TP8: TestPoint, symbol Connector:TestPoint
- added U87: SN74LVC1T45DBV, Package_TO_SOT_SMD:SOT-23-6, symbol Logic_LevelTranslator:SN74LVC1T45DBV
Connections:
- new net: R9.1, U87.3 (A)
- new net +3.3V: C41.1, U87.1 (VCCA), U87.5 (DIR)
- new net +5V_LED: C42.1, U87.6 (VCCB)
- new net GND: C41.2, C42.2, U87.2 (GND)
- new net LED00: TP8.1, U87.4 (B)
- new net LED_TEST_POINT: TP1.1
- new net RGB_DAT: R9.2
Other:
- added sheet led (led.kicad_sch)
- added sheet led1 (led.kicad_sch)
- added sheet led10 (led.kicad_sch)
- added sheet led11 (led.kicad_sch)
- added sheet led12 (led.kicad_sch)
- added sheet led13 (led.kicad_sch)
- added sheet led14 (led.kicad_sch)
- added sheet led15 (led.kicad_sch)
- added sheet led16 (led.kicad_sch)
- added sheet led17 (led.kicad_sch)
- added sheet led18 (led.kicad_sch)
- added sheet led19 (led.kicad_sch)
- added sheet led2 (led.kicad_sch)
- added sheet led20 (led.kicad_sch)
- added sheet led21 (led.kicad_sch)
- added sheet led22 (led.kicad_sch)
- added sheet led23 (led.kicad_sch)
- added sheet led24 (led.kicad_sch)
- added sheet led25 (led.kicad_sch)
- added sheet led26 (led.kicad_sch)
- added sheet led27 (led.kicad_sch)
- added sheet led28 (led.kicad_sch)
- added sheet led29 (led.kicad_sch)
- added sheet led3 (led.kicad_sch)
- added sheet led30 (led.kicad_sch)
- added sheet led31 (led.kicad_sch)
- added sheet led32 (led.kicad_sch)
- added sheet led33 (led.kicad_sch)
- added sheet led34 (led.kicad_sch)
- added sheet led35 (led.kicad_sch)
- added sheet led36 (led.kicad_sch)
- added sheet led37 (led.kicad_sch)
- added sheet led38 (led.kicad_sch)
- added sheet led39 (led.kicad_sch)
- added sheet led4 (led.kicad_sch)
- added sheet led40 (led.kicad_sch)
- added sheet led41 (led.kicad_sch)
- added sheet led42 (led.kicad_sch)
- added sheet led43 (led.kicad_sch)
- added sheet led44 (led.kicad_sch)
- added sheet led45 (led.kicad_sch)
- added sheet led46 (led.kicad_sch)
- added sheet led47 (led.kicad_sch)
- added sheet led48 (led.kicad_sch)
- added sheet led49 (led.kicad_sch)
- added sheet led5 (led.kicad_sch)
- added sheet led50 (led.kicad_sch)
- added sheet led51 (led.kicad_sch)
- added sheet led52 (led.kicad_sch)
- added sheet led53 (led.kicad_sch)
- added sheet led54 (led.kicad_sch)
- added sheet led55 (led.kicad_sch)
- added sheet led56 (led.kicad_sch)
- added sheet led57 (led.kicad_sch)
- added sheet led58 (led.kicad_sch)
- added sheet led59 (led.kicad_sch)
- added sheet led6 (led.kicad_sch)
- added sheet led60 (led.kicad_sch)
- added sheet led61 (led.kicad_sch)
- added sheet led62 (led.kicad_sch)
- added sheet led63 (led.kicad_sch)
- added sheet led64 (led.kicad_sch)
- added sheet led65 (led.kicad_sch)
- added sheet led66 (led.kicad_sch)
- added sheet led67 (led.kicad_sch)
- added sheet led68 (led.kicad_sch)
- added sheet led69 (led.kicad_sch)
- added sheet led7 (led.kicad_sch)
- added sheet led70 (led.kicad_sch)
- added sheet led71 (led.kicad_sch)
- added sheet led72 (led.kicad_sch)
- added sheet led73 (led.kicad_sch)
- added sheet led74 (led.kicad_sch)
- added sheet led75 (led.kicad_sch)
- added sheet led76 (led.kicad_sch)
- added sheet led8 (led.kicad_sch)
- added sheet led9 (led.kicad_sch)
- note added: "RGB = TIM1_CH1 + DMA background; never in 125 µs scan loop. Inject +5V_LED at multiple points; bulk 100-470 µF at injection. Keep RGB power/switching away from analog front end; separate returns."
