File: kicad/display.kicad_sch (KiCad schematic)
At the start: 0 parts

Commit message: finish schematics
Parts:
- added J2: Conn_01x08, symbol Connector_Generic:Conn_01x08
Connections:
- new net +3.3V: J2.2 (Pin_2)
- new net DISP_BLK: J2.8 (Pin_8)
- new net DISP_CS: J2.7 (Pin_7)
- new net DISP_DC: J2.6 (Pin_6)
- new net DISP_RES: J2.5 (Pin_5)
- new net DISP_SCL: J2.3 (Pin_3)
- new net DISP_SDA: J2.4 (Pin_4)
- new net GND: J2.1 (Pin_1)
