File: kicad/power.kicad_sch (KiCad schematic)
At the start: 33 parts, among them U1 AP2112K-3.3, U2 TPS7A20xxxDBV

Commit message: finish schematics
Parts:
- added TP2, TP3, TP4, TP5, TP6, TP7: TestPoint, symbol Connector:TestPoint
Connections:
- net +3.3V: now also TP2.1
- net +3.3VA: now also TP3.1
- net GND: now also TP6.1
- net GNDA: now also TP7.1
- net +5VLED renamed +5V_LED
- net +5V_LED: now also TP4.1, TP5.1
Other:
- note added: "Test Points"
